File: Flight Controller/ASTRA.kicad_pcb (KiCad board)
At the start: 2 copper layers, 74 x 77.5 mm, 34 parts

Commit message: a lil tweak on the pcb
Routing:
- net /CE: track 37.4 -> 34.7 mm
- net /SERVO4: track 21.2 -> 20.0 mm
- net /SERVO3: track 16.3 -> 15.5 mm
- net /SERVO1: track 12.2 -> 13.0 mm
- net /CSN: track 28.6 -> 28.0 mm
Changed lines of the file:
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@@
 			(drillshape 0)
 			(scaleselection 1)
-			(outputdirectory "../../akakakkak/AAAgerber/")
+			(outputdirectory "../../ASTRA_GERBER/")
 		)
 	)
@@
 	)
 	(segment
-		(start 119.06 104.695)
-		(end 122.44 104.695)
+		(start 123.105 104.695)
+		(end 123.4 104.4)
 		(width 0.2)
 		(layer "F.Cu")
@@
 	)
 	(segment
-		(start 122.44 104.695)
-		(end 122.46 104.675)
+		(start 129.085 90.9)
+		(end 143.42 90.9)
 		(width 0.2)
 		(layer "F.Cu")
@@
 	)
 	(segment
-		(start 129.085 90.9)
-		(end 143.42 90.9)
+		(start 119.06 104.695)
+		(end 123.105 104.695)
 		(width 0.2)
 		(layer "F.Cu")
@@
 	)
 	(via
-		(at 129.06 90.875)
+		(at 123.4 104.4)
 		(size 0.6)
 		(drill 0.3)
@@
 	)
 	(via
-		(at 122.46 104.675)
+		(at 129.06 90.875)
 		(size 0.6)
 		(drill 0.3)
@@
 	)
 	(segment
-		(start 123.86 90.875)
+		(start 123.4 96.535)
 		(end 129.06 90.875)
 		(width 0.2)
@@
 	)
 	(segment
-		(start 122.46 104.675)
-		(end 123.66 103.475)
-		(width 0.2)
-		(layer "B.Cu")
-		(net 6)
-	)
-	(segment
-		(start 123.66 103.475)
-		(end 123.66 91.075)
-		(width 0.2)
-		(layer "B.Cu")
-		(net 6)
-	)
-	(segment
-		(start 123.66 91.075)
-		(end 123.86 90.875)
+		(start 123.4 104.4)
+		(end 123.4 96.535)
 		(width 0.2)
 		(layer "B.Cu")
@@
 	)
 	(segment
-		(start 172.25 92.75)
-		(end 167.25 97.75)
-		(width 0.2)
-		(layer "F.Cu")
-		(net 11)
-	)
-	(segment
-		(start 167.25 97.75)
-		(end 167.25 99.75)
-		(width 0.2)
-		(layer "F.Cu")
-		(net 11)
-	)
-	(segment
-		(start 167.25 99.75)
-		(end 165.94 101.06)
-		(width 0.2)
-		(layer "F.Cu")
-		(net 11)
-	)
-	(segment
 		(start 165.94 101.06)
 		(end 162 101.06)
@@
 	(segment
 		(start 173.71 92.75)
-		(end 172.25 92.75)
+		(end 173.71 93.29)
 		(width 0.2)
 		(layer "F.Cu")
@@
 	)
 	(segment
-		(start 173.75 84.825)
-		(end 171.675 84.825)
+		(start 173.71 93.29)
+		(end 165.94 101.06)
 		(width 0.2)
 		(layer "F.Cu")
-		(net 12)
+		(net 11)
 	)
 	(segment
-		(start 171.675 84.825)
-		(end 167.25 89.25)
+		(start 173.75 84.825)
+		(end 167.25 91.325)
 		(width 0.2)
 		(layer "F.Cu")
@@
 	)
 	(segment
-		(start 167.25 89.25)
+		(start 167.25 91.325)
 		(end 167.25 95.75)
 		(width 0.2)
@@
 	)
 	(segment
-		(start 119.06 102.155)
-		(end 126.14 102.155)
+		(start 135.16 93.44)
+		(end 143.42 93.44)
 		(width 0.2)
 		(layer "F.Cu")
@@
 	)
 	(segment
-		(start 126.14 102.155)
-		(end 126.66 102.675)
+		(start 126.245 102.155)
+		(end 126.6 101.8)
 		(width 0.2)
 		(layer "F.Cu")
@@
 	)
 	(segment
-		(start 138.695 93.44)
-		(end 143.42 93.44)
+		(start 119.06 102.155)
+		(end 126.245 102.155)
 		(width 0.2)
 		(layer "F.Cu")
@@
 	)
 	(segment
-		(start 138.66 93.475)
-		(end 138.695 93.44)
+		(start 135 93.6)
+		(end 135.16 93.44)
 		(width 0.2)
 		(layer "F.Cu")
@@
 	)
 	(via
-		(at 138.66 93.475)
+		(at 135 93.6)
 		(size 0.6)
 		(drill 0.3)
@@
 	)
 	(via
-		(at 126.66 102.675)
+		(at 126.6 101.8)
 		(size 0.6)
 		(drill 0.3)
@@
 	)
 	(segment
-		(start 127.86 102.875)
-		(end 137.26 93.475)
+		(start 126.6 101.8)
+		(end 134.8 93.6)
 		(width 0.2)
 		(layer "B.Cu")
@@
 	)
 	(segment
-		(start 126.66 102.675)
-		(end 126.86 102.875)
-		(width 0.2)
-		(layer "B.Cu")
-		(net 21)
-	)
-	(segment
-		(start 126.86 102.875)
-		(end 127.86 102.875)
-		(width 0.2)
-		(layer "B.Cu")
-		(net 21)
-	)
-	(segment
-		(start 137.26 93.475)
-		(end 138.66 93.475)
+		(start 134.8 93.6)
+		(end 135 93.6)
 		(width 0.2)
 		(layer "B.Cu")
@@
 	)
 	(segment
-		(start 170 108.5)
-		(end 167.64 106.14)
+		(start 170.74 106.14)
+		(end 161.2 106.14)
 		(width 0.2)
 		(layer "F.Cu")
@@
 	(segment
 		(start 173.21 108.5)
-		(end 170 108.5)
+		(end 173.1 108.5)
 		(width 0.2)
 		(layer "F.Cu")
@@
 	)
 	(segment
-		(start 167.64 106.14)
-		(end 162 106.14)
+		(start 173.1 108.5)
+		(end 170.74 106.14)
 		(width 0.2)
 		(layer "F.Cu")
@@
 	)
 	(segment
-		(start 168.4 103.6)
-		(end 162 103.6)
+		(start 173.5 100.575)
+		(end 173.425 100.575)
 		(width 0.2)
 		(layer "F.Cu")
@@
 	)
 	(segment
-		(start 171.425 100.575)
-		(end 168.4 103.6)
+		(start 173.425 100.575)
+		(end 170.4 103.6)
 		(width 0.2)
 		(layer "F.Cu")
@@
 	)
 	(segment
-		(start 173.5 100.575)
-		(end 171.425 100.575)
+		(start 170.4 103.6)
+		(end 162 103.6)
 		(width 0.2)
 		(layer "F.Cu")
