File: Flight Controller/ASTRA.kicad_sch (KiCad schematic)
At the start: 30 parts

Commit message: a lil tweak on the pcb
Changed lines of the file:
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@@
 		(on_board yes)
 		(dnp no)
-		(fields_autoplaced yes)
 		(property "Reference" "C11"
-			(at 88.9 81.2799 0)
+			(at 77.724 80.01 0)
 			(effects
 				(font
@@
 		)
 		(property "Value" "0.1uf"
-			(at 88.9 83.8199 0)
+			(at 76.962 82.296 0)
 			(effects
 				(font
@@
 		(on_board yes)
 		(dnp no)
-		(fields_autoplaced yes)
 		(property "Reference" "C13"
-			(at 88.9 102.8699 0)
+			(at 77.724 101.6 0)
 			(effects
 				(font
@@
 		)
 		(property "Value" "0.1uf"
-			(at 88.9 105.4099 0)
+			(at 77.216 103.886 0)
 			(effects
 				(font
@@
 		(on_board yes)
 		(dnp no)
-		(fields_autoplaced yes)
 		(property "Reference" "C17"
-			(at 199.39 125.7299 0)
+			(at 188.468 124.714 0)
 			(effects
 				(font
@@
 		)
 		(property "Value" "0.1uf"
-			(at 199.39 128.2699 0)
+			(at 187.706 127.254 0)
 			(effects
 				(font
@@
 		(on_board yes)
 		(dnp no)
-		(fields_autoplaced yes)
 		(property "Reference" "C14"
-			(at 99.06 148.5899 0)
+			(at 88.9 145.034 0)
 			(effects
 				(font
@@
 		)
 		(property "Value" "0.1uf"
-			(at 99.06 151.1299 0)
+			(at 88.392 147.574 0)
 			(effects
 				(font
@@
 		(on_board yes)
 		(dnp no)
-		(fields_autoplaced yes)
 		(property "Reference" "C18"
-			(at 199.39 110.4899 0)
+			(at 188.214 109.474 0)
 			(effects
 				(font
@@
 		)
 		(property "Value" "0.1uf"
-			(at 199.39 113.0299 0)
+			(at 187.452 111.76 0)
 			(effects
 				(font
@@
 		(on_board yes)
 		(dnp no)
-		(fields_autoplaced yes)
 		(property "Reference" "C15"
-			(at 99.06 163.8299 0)
+			(at 88.392 160.782 0)
 			(effects
 				(font
@@
 		)
 		(property "Value" "0.1uf"
-			(at 99.06 166.3699 0)
+			(at 87.884 163.068 0)
 			(effects
 				(font
@@
 		(on_board yes)
 		(dnp no)
-		(fields_autoplaced yes)
 		(property "Reference" "C19"
-			(at 199.39 96.5199 0)
+			(at 188.214 95.504 0)
 			(effects
 				(font
@@
 		)
 		(property "Value" "0.1uf"
-			(at 199.39 99.0599 0)
+			(at 187.706 98.044 0)
 			(effects
 				(font
@@
 		(on_board yes)
 		(dnp no)
-		(fields_autoplaced yes)
 		(property "Reference" "C16"
-			(at 199.39 143.5099 0)
+			(at 187.706 141.986 0)
 			(effects
 				(font
@@
 		)
 		(property "Value" "0.1uf"
-			(at 199.39 146.0499 0)
+			(at 187.198 144.272 0)
 			(effects
 				(font
@@
 		(on_board yes)
 		(dnp no)
-		(fields_autoplaced yes)
 		(property "Reference" "C12"
-			(at 88.9 60.9599 0)
+			(at 76.962 59.69 0)
 			(effects
 				(font
@@
 		)
 		(property "Value" "0.1uf"
-			(at 88.9 63.4999 0)
-			(effects
-				(font
+			(at 76.454 61.976 0)
+			(effects
+				(font
