File: FlightController/ASTRA.kicad_sch (KiCad schematic)
At the start: 38 parts

Commit message: added new flight controller pcb files
Parts:
- added C6: 100uf, Capacitor_THT:CP_Radial_D6.3mm_P2.50mm, symbol Device:C
- C1: footprint Capacitor_THT:CP_Radial_D5.0mm_P2.00mm -> Capacitor_THT:CP_Radial_D10.0mm_P5.00mm
- C3, C4, C5: footprint Capacitor_THT:CP_Radial_D5.0mm_P2.00mm -> Capacitor_THT:CP_Radial_D6.3mm_P2.50mm
Connections:
- net 5V: now also C6.1
- net CE: now also A1.19 (GPIO14); no longer A1.11 (GPIO8)
- net CSN: now also A1.20 (GPIO15); no longer A1.12 (GPIO9)
- net GND: now also C6.2
- net MISO: now also A1.6 (GPIO4); no longer A1.16 (GPIO12)
- net MOSI: now also A1.10 (GPIO7); no longer A1.15 (GPIO11)
- net RCV_L2: now also A1.11 (GPIO8); no longer A1.6 (GPIO4)
- net SCK: now also A1.9 (GPIO6); no longer A1.14 (GPIO10)
- net SERVO5_LGT: now also A1.5 (GPIO3); no longer A1.20 (GPIO15)
- net SERVO6_SLN: now also A1.4 (GPIO2); no longer A1.19 (GPIO14)
- net SERVO7_TVM: now also A1.15 (GPIO11); no longer A1.10 (GPIO7)
- net SERVO8_TVM: now also A1.14 (GPIO10); no longer A1.9 (GPIO6)
- net XMIT_L2: now also A1.12 (GPIO9); no longer A1.7 (GPIO5)
- net GPIO_NCH: no longer names the net of A1.17 (GPIO13)
- net GPIO_SLN: no longer names the net of A1.29 (GPIO22)
Changed lines of the file:
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@@
 	)
 	(label "SERVO7_TVM"
-		(at 118.11 114.3 180)
+		(at 118.11 124.46 180)
 		(effects
 			(font
@@
 	)
 	(label "SERVO6_SLN"
-		(at 118.11 132.08 180)
+		(at 118.11 101.6 180)
 		(effects
 			(font
@@
 		)
 	)
-	(label "GPIO_SLN"
-		(at 163.83 114.3 0)
-		(effects
-			(font
-				(size 1.27 1.27)
-			)
-			(justify left bottom)
-		)
-	)
 	(label "GND"
 		(at 128.27 69.85 90)
@@
 	)
 	(label "MOSI"
-		(at 118.11 124.46 180)
+		(at 118.11 114.3 180)
 		(effects
 			(font
@@
 		)
 	)
+	(label "GND"
+		(at 233.68 86.36 0)
+		(effects
+			(font
+				(size 1.27 1.27)
+			)
+			(justify left bottom)
+		)
+	)
 	(label "5V"
 		(at 193.04 59.69 180)
@@
 	)
 	(label "XMIT_L2"
-		(at 118.11 109.22 180)
+		(at 118.11 119.38 180)
 		(effects
 			(font
@@
 	)
 	(label "SERVO8_TVM"
-		(at 118.11 111.76 180)
+		(at 118.11 121.92 180)
 		(effects
 			(font
@@
 	)
 	(label "CSN"
-		(at 118.11 119.38 180)
+		(at 118.11 134.62 180)
 		(effects
 			(font
@@
 	)
 	(label "CE"
-		(at 118.11 116.84 180)
+		(at 118.11 132.08 180)
 		(effects
 			(font
@@
 	)
 	(label "SERVO5_LGT"
-		(at 118.11 134.62 180)
+		(at 118.11 104.14 180)
 		(effects
 			(font
@@
 	)
 	(label "MISO"
-		(at 118.11 127 180)
+		(at 118.11 106.68 180)
 		(effects
 			(font
@@
 		)
 	)
-	(label "GPIO_NCH"
-		(at 118.11 129.54 180)
-		(effects
-			(font
-				(size 1.27 1.27)
-			)
-			(justify right bottom)
-		)
-	)
 	(label "5V"
 		(at 260.35 58.42 270)
@@
 	)
 	(label "SCK"
-		(at 118.11 121.92 180)
+		(at 118.11 111.76 180)
 		(effects
 			(font
@@
 		)
 	)
+	(label "5V"
+		(at 233.68 93.98 270)
+		(effects
+			(font
+				(size 1.27 1.27)
+			)
+			(justify right bottom)
+		)
+	)
 	(label "GND"
 		(at 95.25 161.29 0)
@@
 	)
 	(label "RCV_L2"
-		(at 118.11 106.68 180)
+		(at 118.11 116.84 180)
 		(effects
 			(font
@@
 			)
 		)
-		(property "Footprint" "Capacitor_THT:CP_Radial_D5.0mm_P2.00mm"
+		(property "Footprint" "Capacitor_THT:CP_Radial_D6.3mm_P2.50mm"
 			(at 239.0648 68.58 0)
 			(effects
@@
 			)
 		)
-		(property "Footprint" "Capacitor_THT:CP_Radial_D5.0mm_P2.00mm"
+		(property "Footprint" "Capacitor_THT:CP_Radial_D6.3mm_P2.50mm"
 			(at 256.8448 81.28 0)
 			(effects
@@
 	)
 	(symbol
+		(lib_id "Device:C")
+		(at 233.68 90.17 180)
+		(unit 1)
+		(exclude_from_sim no)
+		(in_bom yes)
+		(on_board yes)
+		(dnp no)
+		(fields_autoplaced yes)
+		(property "Reference" "C6"
+			(at 237.49 88.8999 0)
+			(effects
+				(font
+					(size 1.27 1.27)
+				)
+				(justify right)
+			)
+		)
+		(property "Value" "100uf"
+			(at 237.49 91.4399 0)
+			(effects
+				(font
+					(size 1.27 1.27)
+				)
+				(justify right)
+			)
+		)
+		(property "Footprint" "Capacitor_THT:CP_Radial_D6.3mm_P2.50mm"
+			(at 232.7148 86.36 0)
+			(effects
+				(font
+					(size 1.27 1.27)
+				)
+				(hide yes)
+			)
+		)
+		(property "Datasheet" "~"
+			(at 233.68 90.17 0)
+			(effects
+				(font
+					(size 1.27 1.27)
+				)
+				(hide yes)
+			)
+		)
+		(property "Description" "Unpolarized capacitor"
+			(at 233.68 90.17 0)
+			(effects
+				(font
+					(size 1.27 1.27)
+				)
+				(hide yes)
+			)
+		)
+		(pin "2"
+		)
+		(pin "1"
+		)
+		(instances
+			(project "ASTRA"
+				(path "/27797d85-b80b-4f85-af9d-7bbd95d91f09"
+					(reference "C6")
+					(unit 1)
+				)
+			)
+		)
+	)
+	(symbol
 		(lib_id "Connector_Generic:Conn_01x02")
 		(at 248.92 35.56 0)
@@
 			)
 		)
-		(property "Footprint" "Capacitor_THT:CP_Radial_D5.0mm_P2.00mm"
+		(property "Footprint" "Capacitor_THT:CP_Radial_D10.0mm_P5.00mm"
 			(at 246.6848 24.13 0)
 			(effects
@@
 			)
 		)
-		(property "Footprint" "Capacitor_THT:CP_Radial_D5.0mm_P2.00mm"
+		(property "Footprint" "Capacitor_THT:CP_Radial_D6.3mm_P2.50mm"
 			(at 259.3848 50.8 0)
 			(effects
